File: PCB/M125/M125.kicad_pcb (KiCad board)
At the start: 2 copper layers, 29 x 13.6 mm, 21 parts, among them J1 Conn_01x04, J2 Conn_01x04, J3 Shelly, Q1 PMF250XNEX, U1 ESP32-PICO-MINI-02, U2 LMR16006+FB

Commit message: Tidy
Other:
- board text added: "${CURRENT_DATE}"
- board text removed: "${DATE}"

Commit message: Library update
Parts:
- removed C3: 100nF, RevK:C_0603_
- removed C4: 2.2uF, RevK:C_0805_
- removed C5: 10uF, RevK:C_0805_
- removed D1: RGB, RevK:LED-RGB-1.6x1.6
- removed D2: Schottky, RevK:D_1206_
- removed L1: 6.8uH, RevK:L_4x4_
- removed R1: 680R, RevK:R_0603
- removed R2: 2K, RevK:R_0603
- removed R3: 220R, RevK:R_0603
- removed R5: 100k 1% or 0R, RevK:R_0603
- removed R6: 30k 1% or NF, RevK:R_0603
- removed U2: LMR16006+FB, RevK:RegulatorBlockFB
- added C6: 10uF 50V, RevK:C_0603_, B.Cu at (82.5, 96.0)
- added C7: 10uF 6.3V, RevK:C_0603_, B.Cu at (82.5, 98.0)
- added C8: 100nF, RevK:C_0603_, B.Cu at (82.5, 99.9)
- added D3: RGB, RevK:LED-RGB-1.6x1.6, B.Cu at (113.0, 90.9)
- added L2: 10uH, RevK:L_4x4_, B.Cu at (81.3, 103.4)
- added PCB1: 70x70, RevK:PCB7070, F.Cu at (100.0, 100.0)
- added R10: 124k, RevK:R_0402_, B.Cu at (82.6, 80.8)
- added R11: 39k2, RevK:R_0402_, B.Cu at (82.6, 82.6)
- added R12: 1M, RevK:R_0402_, B.Cu at (82.6, 84.5)
- added R7: 680R, RevK:R_0402, B.Cu at (113.0, 92.6)
- added R8: 2K, RevK:R_0402, B.Cu at (112.2, 92.6)
- added R9: 220R, RevK:R_0402, B.Cu at (113.8, 92.6)
- added U3: MD8942, RevK:SOT-23-6-MD8942, B.Cu at (100.0, 97.3)
- added V1: ~, RevK:VCUT70, F.Cu at (100.0, 89.0)
- added V2: ~, RevK:VCUT70, F.Cu at (100.0, 100.8)
- C1: value 10nF -> 1uF; footprint RevK:C_0603 -> RevK:C_0402
- C2: footprint RevK:C_0603 -> RevK:C_0402
- J1, J2: footprint RevK:Molex_MiniSPOX_H4RA -> RevK:PTSM-HH-4-RA
- R4: footprint RevK:R_0603 -> RevK:R_0402
- moved Logo1 58.7 mm to (111.2, 97.7)
- moved C2 51.0 mm to (93.9, 91.3)
- moved U1 50.7 mm to (100.0, 94.9)
- moved Q1 49.4 mm to (89.8, 98.9)
- moved J1 49.0 mm to (92.1, 94.9)
- moved J2 49.0 mm to (107.9, 94.9)
- moved C1 49.0 mm to (95.3, 96.2)
- moved R4 49.0 mm to (94.9, 92.0)
- moved J3 45.7 mm to (87.2, 94.9), turned to 90 degrees
Connections:
- J1 pad 4: Net-(J1-Pad4) -> Net-(J1-Pin_4)
- Q1 pad 1: Net-(J1-Pad4) -> SEND
- Q1 pad 3: SEND -> Net-(J1-Pin_4)
Routing:
- net +3V3: track 41.0 -> 0.00 mm, vias 1 -> 0
- net SEND: track 10.8 -> 0.00 mm, vias 1 -> 0
- net TX: track 9.52 -> 0.00 mm, vias 1 -> 0
- net B: track 9.13 -> 0.00 mm, vias 1 -> 0
- net RX: track 8.70 -> 0.00 mm, vias 1 -> 0
- net G: track 8.58 -> 0.00 mm, vias 1 -> 0
- net GPIO0: track 7.65 -> 0.00 mm
- net DC: track 7.18 -> 0.00 mm
- net NFCTX: track 7.13 -> 0.00 mm
- net R: track 6.46 -> 0.00 mm, vias 1 -> 0
- net Net-(D1-Pad3): track 6.08 -> 0.00 mm
- net EN: track 4.58 -> 0.00 mm, vias 1 -> 0
- net DATA: track 4.55 -> 0.00 mm, vias 1 -> 0
- net Net-(D1-Pad4): track 4.53 -> 0.00 mm
- net GND: track 4.46 -> 0.00 mm, vias 1 -> 0
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Other:
- board size 29 x 13.6 mm -> 70 x 70 mm

Commit message: PCB Update
Parts:
- C6: value 10uF 50V -> 10uF 35V
