File: PCB/M125/M125.kicad_sch (KiCad schematic)
At the start: 21 parts, among them J1 Conn_01x04, J2 Conn_01x04, J3 Shelly, Q1 PMF250XNEX, U1 ESP32-PICO-MINI-02, U2 LMR16006+FB

Commit message: Library update
Parts:
- removed C3: 100nF, RevK:C_0603_, symbol RevK:Hidden
- removed C4: 2.2uF, RevK:C_0805_, symbol RevK:Hidden
- removed C5: 10uF, RevK:C_0805_, symbol RevK:Hidden
- removed D1: RGB, RevK:LED-RGB-1.6x1.6, symbol Device:LED_ARGB
- removed D2: Schottky, RevK:D_1206_, symbol RevK:Hidden
- removed L1: 6.8uH, RevK:L_4x4_, symbol RevK:Hidden
- removed R1: 680R, RevK:R_0603, symbol Device:R
- removed R2: 2K, RevK:R_0603, symbol Device:R
- removed R3: 220R, RevK:R_0603, symbol Device:R
- removed R5: 100k 1% or 0R, RevK:R_0603, symbol Device:R
- removed R6: 30k 1% or NF, RevK:R_0603, symbol Device:R
- removed U2: LMR16006+FB, RevK:RegulatorBlockFB, symbol RevK:LMR16006+FB
- added C6: 10uF 50V, RevK:C_0603_, symbol RevK:Hidden
- added C7: 10uF 6.3V, RevK:C_0603_, symbol RevK:Hidden
- added C8: 100nF, RevK:C_0603_, symbol RevK:Hidden
- added D3: RGB, RevK:LED-RGB-1.6x1.6, symbol Device:LED_RGBA
- added L2: 10uH, RevK:L_4x4_, symbol RevK:Hidden
- added PCB1: 70x70, RevK:PCB7070, symbol RevK:PCB
- added R10: 124k, RevK:R_0402_, symbol RevK:Hidden
- added R11: 39k2, RevK:R_0402_, symbol RevK:Hidden
- added R12: 1M, RevK:R_0402_, symbol RevK:Hidden
- added R7: 680R, RevK:R_0402, symbol Device:R
- added R8: 2K, RevK:R_0402, symbol Device:R
- added R9: 220R, RevK:R_0402, symbol Device:R
- added U3: MD8942, RevK:SOT-23-6-MD8942, symbol RevK:MD89420-RegBlock
- added V1, V2: ~, RevK:VCUT70, symbol RevK:VCUT
- C1: value 10nF -> 1uF; footprint RevK:C_0603 -> RevK:C_0402
- C2: footprint RevK:C_0603 -> RevK:C_0402
- J1, J2: footprint RevK:Molex_MiniSPOX_H4RA -> RevK:PTSM-HH-4-RA
- R4: footprint RevK:R_0603 -> RevK:R_0402
Connections:
- net +3V3: now also D3.4 (A), U3.8 (VOUT)
- net B: now also R9.2
- net DC: now also U3.5 (VIN)
- net G: now also R8.2
- net GND: now also U3.2 (GND), U3.7 (GND)
- net R: now also R7.2
- net SEND: now also Q1.1 (G); no longer Q1.3 (D)
- net at J1.4 (Pin_4): now also Q1.3 (D); no longer Q1.1 (G)
- new net: D3.1 (RK), R7.1
- new net: D3.2 (GK), R8.1
- new net: D3.3 (BK), R9.1
- no-connect marks 17 -> 18
Other:
- moved on the sheet: J1, Q1

Commit message: PCB Update
Parts:
- C6: value 10uF 50V -> 10uF 35V; LCSC Part # C1591 -> (none); MPN (none) -> C194427
- C7: LCSC Part # C1691 -> (none); MPN (none) -> C1691
- D3: LCSC Part # C264508 -> (none); MPN (none) -> C264508
- U3: LCSC Part # C2684786 -> (none); MPN (none) -> C2684786
Changed lines of the file:
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@@
       (effects (font (size 1.27 1.27)) hide)
     )
-    (property "LCSC Part #" "C2684786" (at 215.265 64.77 0)
+    (property "MPN" "C2684786" (at 215.265 64.77 0)
       (effects (font (size 1.27 1.27)) hide)
     )
@@
       (effects (font (size 1.27 1.27)) hide)
     )
-    (property "LCSC Part #" "C264508" (at 69.85 122.555 0)
+    (property "MPN" "C264508" (at 69.85 122.555 0)
       (effects (font (size 1.27 1.27)) hide)
     )
@@
       (effects (font (size 1.27 1.27)) (justify left))
     )
-    (property "Value" "10uF 50V" (at 242.57 31.75 0)
+    (property "Value" "10uF 35V" (at 242.57 31.75 0)
       (effects (font (size 1.27 1.27)) (justify left))
     )
@@
       (effects (font (size 1.27 1.27)) hide)
     )
-    (property "LCSC Part #" "C1591" (at 236.22 31.75 0)
+    (property "MPN" "C194427" (at 236.22 31.75 0)
       (effects (font (size 1.27 1.27)) hide)
     )
@@
       (effects (font (size 1.27 1.27)) hide)
     )
-    (property "LCSC Part #" "C1691" (at 236.22 33.655 0)
-      (effects (font (size 1.27 1.27)) hide)
-    )
+    (property "MPN" "C1691" (at 236.22 33.655 0)
+      (effects (font (size 1.27 1.27)) hide)
+    )
